Commit message: ajout du second finger

File: urdf/finger.urdl.xacro (robot description, xacro)
@@ -1,9 +1,17 @@
 <?xml version="1.0"?>
 <robot xmlns:xacro="http://ros.org/wiki/xacro" name="finger">
-    <xacro:macro name="finger" params="parent prefix joint_type">
-        <link name="${prefix}_link" />
-        <joint name="${prefix}_joint" type="${joint_type}">
+    <xacro:macro name="finger" params="parent prefix lower upper">
+        <link name="${prefix}_link">
+            <visual>
+            <geometry>
+                <mesh filename="file:///$(find robot_nano_hand_teleop)/models/robot_nano_hand_${prefix}_link1.stl" scale="1 1 1"/>
+            <geometry>
+            <material name="green"/>
+            </visual>
+        </link>
+        <joint name="${prefix}_joint" type="revolute">
             <parent link="${parent}" />
             <child link="${prefix}_link" />
+            <limit lower=${lower} upper=${upper} />
         </joint>
     </xacro:macro>
